File: Arduino DC-DC Converter Control Board.kicad_pcb (KiCad board)
At the start: 2 copper layers, 100 x 68 mm, 31 parts, among them J3 Arduino VIN_Enable, J5 Pick 3.3V or GND, J7 Load Resistor Socket, Q1 IRF9640, Q2 2N2222

Commit message: Added LTspice files.
Parts:
- C3: value CP1 -> 100uF
- D1: footprint Diode_SMD:D_SMA -> Diode_SMD:D_3220_8050Metric
- moved D1 3.42 mm to (72.8, 50.9)
Routing:
- net Net-(D1-Pad1): track 30.9 -> 36.2 mm
- net GND: track 164.7 -> 165.9 mm, vias 1 -> 2
