File: Arduino DC-DC Converter Control Board.sch (KiCad schematic (older format))
At the start: 31 parts, among them J3 Arduino VIN_Enable, J5 Pick 3.3V or GND, J7 Load Resistor Socket, Q1 IRF9640, Q2 2N2222

Commit message: Added LTspice files.
Parts:
- D1: footprint Diode_SMD:D_SMA -> Diode_SMD:D_3220_8050Metric; Digikey https://www.diodes.com/assets/Datasheets/ds13012.pdf -> https://www.digikey.com/en/products/detail/diodes-incorpora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
Changed lines of the file:
@@
 Title "Arduino DC-DC Converter Control Board "
 Date "2021-02-05"
-Rev "0.11"
+Rev "0.111"
 Comp "Walla Walla University"
 Comment1 "Rob Frohne"
 Comment2 "This board is for experiments with controlling a DC-DC  converter using an Arduino."
-Comment3 ""
+Comment3 "Fixed the footprint of D1"
 Comment4 ""
 $EndDescr
@@
 F 0 "D1" V 4104 1930 50  0000 L CNN
 F 1 "B540C" V 4195 1930 50  0000 L CNN
-F 2 "Diode_SMD:D_SMA" H 4150 1850 50  0001 C CNN
+F 2 "Diode_SMD:D_3220_8050Metric" H 4150 1850 50  0001 C CNN
 F 3 "https://www.diodes.com/assets/Datasheets/ds13012.pdf" H 4150 1850 50  0001 C CNN
-F 4 "https://www.diodes.com/assets/Datasheets/ds13012.pdf" V 4150 1850 50  0001 C CNN "Digikey"
+F 4 "https://www.digikey.com/en/products/detail/diodes-incorporated/B540C-13-F/768771" V 4150 1850 50  0001 C CNN "Digikey"
 	1    4150 1850
 	0    1    1    0
